File: PCB files/The Extender PCB.sch (EAGLE design)
At the start: 110 parts, among them J2 AVR_SPI_PROG_3X2NS, U2 328P, Y1 16MHz

Commit message: Redesigned the PCB for the final matrix size
It's now 5x15, the controller was changed to a Teensy 2.0 istead of an AtMEGA 328P
Parts:
- removed C1: 4.7u, adafruit:CPOL-USE2.5-5
- removed C2, C3: 100n, adafruit:C-US050-025X075
- removed C4, C5: 20p, adafruit:C-US050-025X075
- removed F1: 72V/0.25A, SparkFun-Fuses:PPTC_PTH
- removed J1: (no value), SparkFun-Connectors:USB_C16PIN
- removed J2: AVR_SPI_PROG_3X2NS, SparkFun-Connectors:AVR_SPI_PROG_3X2NS
- removed J3: (no value), SparkFun-Connectors:CONN_04
- removed R1: 1.5k, adafruit:R-US_0207/7
- removed R2, R3: 75R, adafruit:R-US_0207/7
- removed R4: 10k, adafruit:R-US_0207/5V
- removed R5, R6: I2C, adafruit:R-US_0207/5V
- removed R7, R8: (no value), adafruit:R-US_0207/5V
- removed S1, S2: MOMENTARY-SWITCH-SPST-PTH-6.0MM, SparkFun-Switches:MOMENTARY-SWITCH-SPST-PTH-6.0MM
- removed SJ1, SJ2: (no value), jumper:SJ
- removed U2: 328P, SparkFun-IC-Microcontroller:ATMEGA328P_PDIP
- removed Y1: 16MHz, SparkFun-Clocks:CRYSTAL-16MHZPTH-HC49US
- added D46, D47, D48, D49, D50, D51, D52, D53, D54, D55, D56, D57, D58, D59, D60, D61, D62, D63, D64, D65, D66, D67, D68, D69, D70, D71, D72, D73, D74, D75: (no value), adafruit:DIODEDO-1N4148
- added LED10, LED11, LED12, LED13, LED14, LED3, LED4, LED5, LED6, LED7, LED8, LED9: WS2812B, SparkFun-LED:WS2812B
- added U$41, U$42, U$43, U$44, U$45, U$46, U$47, U$48, U$49, U$50, U$51, U$52, U$53, U$54, U$55, U$56, U$57, U$58, U$59, U$60, U$61, U$62, U$63, U$64, U$65, U$66, U$67, U$68, U$69, U$70, U$71, U$72, U$73, U$74, U$75: CHERRY-MX1A-E1NW-LED, my_parts:CHERRY-MX1A-E1NW-LED
- added _1: TEENSY, teensy:TEENSY
- D41, D42, D43: value WS2812B -> (none); device SparkFun-LED:WS2812B -> adafruit:DIODEDO-1N4148
- D44, D45: value 3.6V -> (none); device adafruit:SCHOTTKY-DIODEDO41-7 -> adafruit:DIODEDO-1N4148
- LED1, LED2: value (none) -> WS2812B; device adafruit:LED3MM -> SparkFun-LED:WS2812B
Connections:
- removed net I2C_SCL: J3.2, R5.1, SJ1.1, U2.PC5(ADC5/SCL)
- removed net I2C_SDA: J3.3, R6.1, SJ2.1, U2.PC4(ADC4/SDA)
- removed net N$43: F1.2, J1.VBUS
- removed net N$44: D44.C, J1.D-, R1.2, R3.2
- removed net N$45: U2.PD0(RXD)
- removed net RESET: J2.5, R4.1, S1.2, U2.PC6(/RESET)
- removed net RGB: LED1.C, LED2.C
- removed net USB_D+: R2.1, U2.PD2(INT0)
- removed net USB_D-: R3.1, U2.PD3(INT1)
- new net COLUMN10: D11.C, D26.C, D41.C, D56.C, D71.C, _1._D7
- new net COLUMN11: D12.C, D27.C, D42.C, D57.C, D72.C, _1._B4
- new net COLUMN12: D13.C, D28.C, D43.C, D58.C, D73.C, _1._B5
- new net COLUMN13: D14.C, D29.C, D44.C, D59.C, D74.C, _1._B6
- new net COLUMN14: D15.C, D30.C, D45.C, D60.C, D75.C, _1._F7
- new net N$113: _1._REF
- new net N$114: _1._F0
- new net N$115: _1._F1
- new net N$116: _1._F4
- new net N$117: _1._F5
- new net N$120: _1._5V2
- new net N$121: _1._RST
- new net N$122: _1._GND1
- new net N$54: D41.A, U$41.A
- new net N$55: D42.A, U$42.A
- new net N$56: D43.A, U$43.A
- new net N$57: D44.A, U$44.A
- new net N$58: D45.A, U$45.A
- new net N$59: D46.A, U$46.A
- new net N$60: D47.A, U$47.A
- new net N$61: D48.A, U$48.A
- new net N$62: D49.A, U$49.A
- new net N$63: D50.A, U$50.A
- new net N$64: D51.A, U$51.A
- new net N$65: D52.A, U$52.A
- new net N$66: D53.A, U$53.A
- new net N$67: D54.A, U$54.A
- new net N$68: D55.A, U$55.A
- new net N$69: D56.A, U$56.A
- new net N$70: D57.A, U$57.A
- new net N$71: D58.A, U$58.A
- new net N$72: D59.A, U$59.A
- new net N$73: D60.A, U$60.A
- new net N$74: D61.A, U$61.A
- new net N$75: D62.A, U$62.A
- new net N$76: D63.A, U$63.A
- new net N$77: D64.A, U$64.A
- new net N$78: D65.A, U$65.A
- new net N$79: D66.A, U$66.A
- new net N$80: D67.A, U$67.A
- new net N$81: D68.A, U$68.A
- new net N$82: D69.A, U$69.A
- new net N$83: D70.A, U$70.A
- new net N$84: D71.A, U$71.A
- new net N$85: D72.A, U$72.A
- new net N$86: D73.A, U$73.A
- new net N$87: D74.A, U$74.A
- new net N$88: D75.A, U$75.A
- new net N$89: LED11.DO, LED12.DI
- new net N$90: LED12.DO, LED13.DI
- new net N$91: LED13.DO, LED14.DI
- new net ROW4: U$61.UP, U$62.UP, U$63.UP, U$64.UP, U$65.UP, U$66.UP, U$67.UP, U$68.UP, U$69.UP, U$70.UP, U$71.UP, U$72.UP, U$73.UP, U$74.UP, U$75.UP
- net 5V: now also LED1.VSS, LED10.VSS, LED11.VSS, LED12.VSS, LED13.VSS, LED14.VSS, LED2.VSS, LED3.VSS, LED4.VSS, LED5.VSS, LED6.VSS, LED7.VSS, LED8.VSS, LED9.VSS, _1.5V; no longer C1.+, C2.1, C3.1, D41.VSS, D42.VSS, D43.VSS, F1.1, J2.2, J3.1, R1.1, R4.2, R5.2, R6.2
- net COLUMN0: now also D16.C, D46.C, D61.C, _1._B7; no longer D11.C, D21.C, U2.PB0(ICP)
- net COLUMN1: now also D17.C, D47.C, D62.C, _1._D0; no longer D12.C, D22.C
- net COLUMN2: now also D18.C, D48.C, D63.C, _1._D1; no longer D13.C, D23.C
- net COLUMN3: now also D19.C, D49.C, D64.C, _1._D2; no longer D14.C, D24.C, S2.1, U2.PD5(T1)
- net COLUMN4: now also D20.C, D50.C, D65.C, _1._D3; no longer D15.C, D25.C, U2.PB2(SS/OC1B)
- net COLUMN5: now also D21.C, D51.C, D66.C, _1._C6; no longer D16.C, D26.C, U2.PB1(OC1A)
- net COLUMN6: now also D22.C, D52.C, D67.C, _1._C7; no longer D17.C, D27.C, U2.PC0(ADC0)
- net COLUMN7: now also D23.C, D53.C, D68.C, _1._D5; no longer D18.C, D28.C, U2.PC1(ADC1)
- net COLUMN8: now also D24.C, D54.C, D69.C, _1._D4; no longer D19.C, D29.C, U2.PC2(ADC2)
- net COLUMN9: now also D25.C, D55.C, D70.C, _1._D6; no longer D20.C, D30.C, U2.PC3(ADC3)
- net GND: now also LED1.VDD, LED10.VDD, LED11.VDD, LED12.VDD, LED13.VDD, LED14.VDD, LED2.VDD, LED3.VDD, LED4.VDD, LED5.VDD, LED6.VDD, LED7.VDD, LED8.VDD, LED9.VDD, U$41.LED-, U$42.LED-, U$43.LED-, U$44.LED-, U$45.LED-, U$46.LED-, U$47.LED-, U$48.LED-, U$49.LED-, U$50.LED-, U$51.LED-, U$52.LED-, U$53.LED-, U$54.LED-, U$55.LED-, U$56.LED-, U$57.LED-, U$58.LED-, U$59.LED-, U$60.LED-, U$61.LED-, U$62.LED-, U$63.LED-, U$64.LED-, U$65.LED-, U$66.LED-, U$67.LED-, U$68.LED-, U$69.LED-, U$70.LED-, U$71.LED-, U$72.LED-, U$73.LED-, U$74.LED-, U$75.LED-, _1._GND; no longer C1.-, C2.2, C3.2, C4.1, C5.1, D41.VDD, D42.VDD, D43.VDD, D44.A, D45.A, J1.GND, J2.6, J3.4, S1.1, S2.2
- net LED+: now also U$41.LED+, U$42.LED+, U$43.LED+, U$44.LED+, U$45.LED+, U$46.LED+, U$47.LED+, U$48.LED+, U$49.LED+, U$50.LED+, U$51.LED+, U$52.LED+, U$53.LED+, U$54.LED+, U$55.LED+, U$56.LED+, U$57.LED+, U$58.LED+, U$59.LED+, U$60.LED+, U$61.LED+, U$62.LED+, U$63.LED+, U$64.LED+, U$65.LED+, U$66.LED+, U$67.LED+, U$68.LED+, U$69.LED+, U$70.LED+, U$71.LED+, U$72.LED+, U$73.LED+, U$74.LED+, U$75.LED+
- net N$41: now also LED1.DO, LED2.DI; no longer D41.DO, D42.DI
- net N$42: now also LED2.DO, LED3.DI; no longer D42.DO, D43.DI
- net N$46: now also LED3.DO, LED4.DI; no longer D45.C, J1.D+, R2.2
- net N$47: now also LED4.DO, LED5.DI; no longer C5.2, U2.PB7(XTAL2/TOSC2), Y1.1
- net N$48: now also LED5.DO, LED6.DI; no longer C4.2, U2.PB6(XTAL1/TOSC1), Y1.2
- net N$49: now also LED6.DO, LED7.DI; no longer R7.1, SJ1.2
- net N$50: now also LED7.DO, LED8.DI; no longer U2.PD1(TXD)
- net N$51: now also LED8.DO, LED9.DI; no longer LED1.A, R7.2
- net N$52: now also LED10.DI, LED9.DO; no longer R8.1, SJ2.2
- net N$53: now also LED10.DO, LED11.DI; no longer LED2.A, R8.2
- net RGB_DATA: now also LED1.DI, _1._F6; no longer D41.DI, U2.PD6(AIN0)
- net ROW0: now also U$11.UP, U$12.UP, U$13.UP, U$14.UP, U$15.UP, _1._B0; no longer J2.1, U2.PB4(MISO)
- net ROW1: now also U$21.UP, U$22.UP, U$23.UP, U$24.UP, U$25.UP, U$26.UP, U$27.UP, U$28.UP, U$29.UP, U$30.UP, _1._B1; no longer J2.3, U$11.UP, U$12.UP, U$13.UP, U$14.UP, U$15.UP, U2.PB5(SCK)
- net ROW2: now also U$31.UP, U$32.UP, U$33.UP, U$34.UP, U$35.UP, U$36.UP, U$37.UP, U$38.UP, U$39.UP, U$40.UP, U$41.UP, U$42.UP, U$43.UP, U$44.UP, U$45.UP, _1._B2; no longer J2.4, U$21.UP, U$22.UP, U$23.UP, U$24.UP, U$25.UP, U$26.UP, U$27.UP, U$28.UP, U$29.UP, U$30.UP, U2.PB3(MOSI/OC2)
- net ROW3: now also U$46.UP, U$47.UP, U$48.UP, U$49.UP, U$50.UP, U$51.UP, U$52.UP, U$53.UP, U$54.UP, U$55.UP, U$56.UP, U$57.UP, U$58.UP, U$59.UP, U$60.UP, _1._B3; no longer U$31.UP, U$32.UP, U$33.UP, U$34.UP, U$35.UP, U$36.UP, U$37.UP, U$38.UP, U$39.UP, U$40.UP, U2.PD4(XCK/T0)
Other:
- moved on the sheet: D11, D12, D13, D14, D15, D16, D17, D18, D19, D20, D21, D22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

Commit message: The first release
This is what you might call the first release. I will order some prototype PCBs with propably a few minor tweeks!
Parts:
- removed _1: TEENSY, teensy:TEENSY
- added C1, C2: 22p, adafruit:C-US025-025X050
- added C3, C4: 0.1u, adafruit:C-US025-025X050
- added C5: 4.7u, adafruit:CPOL-USE2-4
- added D76, D77: (no value), diode:ZENER-DIODEDO34-7
- added F1: 72V/0.25A, SparkFun-Fuses:PPTC_PTH
- added IC1: ATMEGA32A-PU, ATMEGA32A-PU:ATMEGA32A-PU
- added ISP1: AVRISP-6, adafruit:AVRISP-6
- added J1: USB4085-GF-A_REVA, USB4085-GF-A_REVA:USB4085-GF-A_REVA
- added LED15: (no value), adafruit:LED3MM
- added R1: 10k, adafruit:R-US_0207/9
- added R2, R7: 1.5k, adafruit:R-US_0207/9
- added R3, R4: 5.1k, adafruit:R-US_0207/9
- added R5, R6: 75R, adafruit:R-US_0207/9
- added S1, S2: (no value), SparkFun-Retired:TAC_SWITCHPTH
- added X1: 49S/18PF, Crystals:49S/18PF
Connections:
- removed net N$113: _1._REF
- removed net N$114: _1._F0
- removed net N$115: _1._F1
- removed net N$116: _1._F4
- removed net N$117: _1._F5
- removed net N$120: _1._5V2
- removed net N$121: _1._RST
- removed net N$122: _1._GND1
- new net BOOT: IC1.PD4_(OC1B), S2.3
- new net LED-: U$1.LED-, U$10.LED-, U$11.LED-, U$12.LED-, U$13.LED-, U$14.LED-, U$15.LED-, U$16.LED-, U$17.LED-, U$18.LED-, U$19.LED-, U$2.LED-, U$20.LED-, U$21.LED-, U$22.LED-, U$23.LED-, U$24.LED-, U$25.LED-, U$26.LED-, U$27.LED-, U$28.LED-, U$29.LED-, U$3.LED-, U$30.LED-, U$31.LED-, U$32.LED-, U$33.LED-, U$34.LED-, U$35.LED-, U$36.LED-, U$37.LED-, U$38.LED-, U$39.LED-, U$4.LED-, U$40.LED-, U$41.LED-, U$42.LED-, U$43.LED-, U$44.LED-, U$45.LED-, U$46.LED-, U$47.LED-, U$48.LED-, U$49.LED-, U$5.LED-, U$50.LED-, U$51.LED-, U$53.LED-, U$54.LED-, U$55.LED-, U$56.LED-, U$57.LED-, U$58.LED-, U$59.LED-, U$6.LED-, U$60.LED-, U$61.LED-, U$62.LED-, U$63.LED-, U$64.LED-, U$65.LED-, U$66.LED-, U$67.LED-, U$68.LED-, U$69.LED-, U$7.LED-, U$71.LED-, U$72.LED-, U$73.LED-, U$74.LED-, U$75.LED-, U$8.LED-, U$9.LED-
- new net LED-\: U$70.LED-
- new net MISO: IC1.PB6_(MISO), ISP1.MISO
- new net MOSI: IC1.PB5_(MOSI), ISP1.MOSI
- new net N$119: U$52.LED-
- new net N$43: C1.2, IC1.XTAL2, X1.2
- new net N$44: C2.2, IC1.XTAL1, X1.1
- new net N$45: LED15.C, R2.1
- new net N$92: J1.GND
- new net N$93: F1.2, J1.VBUS
- new net N$94: J1.SHELL
- new net N$95: J1.CC1, R3.1
- new net N$96: D76.C, J1.DN1, J1.DN2, R5.1, R7.1
- new net N$97: D77.C, J1.DP1, J1.DP2, R6.1
- new net N$98: J1.CC2, R4.1
- new net RESET: IC1.!RESET, ISP1.RST, R1.1, S1.3
- new net SCK: IC1.PB7_(SCK), ISP1.SCK
- new net USB_D+: IC1.PD2_(INT0), R6.2
- new net USB_D-: IC1.PD3_(INT1), R5.2
- net 5V: now also C3.1, C4.1, C5.+, F1.1, IC1.AVCC, IC1.VCC, ISP1.VCC, LED15.A, R1.2, R7.2; no longer _1.5V
- net COLUMN0: now also IC1.PD0_(RXD); no longer _1._B7
- net COLUMN1: now also IC1.PD1_(TXD); no longer _1._D0
- net COLUMN10: now also IC1.PA6_(ADC6); no longer _1._D7
- net COLUMN11: now also IC1.PA7_(ADC7); no longer _1._B4
- net COLUMN12: now also IC1.AREF; no longer _1._B5
- net COLUMN13: now also IC1.PC7_(TOSC2); no longer _1._B6
- net COLUMN14: now also IC1.PC6_(TOSC1); no longer _1._F7
- net COLUMN2: now also IC1.PD5_(OC1A); no longer _1._D1
- net COLUMN3: now also IC1.PD6_(ICP1); no longer _1._D2
- net COLUMN4: now also IC1.PA0_(ADC0); no longer _1._D3
- net COLUMN5: now also IC1.PA1_(ADC1); no longer _1._C6
- net COLUMN6: now also IC1.PA2_(ADC2); no longer _1._C7
- net COLUMN7: now also IC1.PA3_(ADC3); no longer _1._D5
- net COLUMN8: now also IC1.PA4_(ADC4); no longer _1._D4
- net COLUMN9: now also IC1.PA5_(ADC5); no longer _1._D6
- net GND: now also C1.1, C2.1, C3.2, C4.2, C5.-, D76.A, D77.A, IC1.GND_1, IC1.GND_2, ISP1.GND, R2.2, R3.2, R4.2, S1.1, S2.1; no longer U$1.LED-, U$10.LED-, U$11.LED-, U$12.LED-, U$13.LED-, U$14.LED-, U$15.LED-, U$16.LED-, U$17.LED-, U$18.LED-, U$19.LED-, U$2.LED-, U$20.LED-, U$21.LED-, U$22.LED-, U$23.LED-, U$24.LED-, U$25.LED-, U$26.LED-, U$27.LED-, U$28.LED-, U$29.LED-, U$3.LED-, U$30.LED-, U$31.LED-, U$32.LED-, U$33.LED-, U$34.LED-, U$35.LED-, U$36.LED-, U$37.LED-, U$38.LED-, U$39.LED-, U$4.LED-, U$40.LED-, U$41.LED-, U$42.LED-, U$43.LED-, U$44.LED-, U$45.LED-, U$46.LED-, U$47.LED-, U$48.LED-, U$49.LED-, U$5.LED-, U$50.LED-, U$51.LED-, U$52.LED-, U$53.LED-, U$54.LED-, U$55.LED-, U$56.LED-, U$57.LED-, U$58.LED-, U$59.LED-, U$6.LED-, U$60.LED-, U$61.LED-, U$62.LED-, U$63.LED-, U$64.LED-, U$65.LED-, U$66.LED-, U$67.LED-, U$68.LED-, U$69.LED-, U$7.LED-, U$70.LED-, U$71.LED-, U$72.LED-, U$73.LED-, U$74.LED-, U$75.LED-, U$8.LED-, U$9.LED-, _1._GND
- net RGB_DATA: now also IC1.PC5_(TDI); no longer _1._F6
- net ROW0: now also IC1.PB0_(XCK/T0); no longer _1._B0
- net ROW1: now also IC1.PB1_(T1); no longer _1._B1
- net ROW2: now also IC1.PB2_(AIN0/INT2); no longer _1._B2
- net ROW3: now also IC1.PB3_(AIN1/OC0); no longer _1._B3
- net ROW4: now also IC1.PB4_(!SS)
