File: PCB files/The Extender PCB.brd (EAGLE design)
At the start: 279.4 x 114.3 mm, 110 parts, among them J2 AVR_SPI_PROG_3X2NS, U2 328P, Y1 16MHz

Commit message: Redesigned the PCB for the final matrix size
It's now 5x15, the controller was changed to a Teensy 2.0 istead of an AtMEGA 328P
Parts:
- removed C1: 4.7u, adafruit:E2,5-5
- removed C2, C3: 100n, adafruit:C050-025X075
- removed C4, C5: 20p, adafruit:C050-025X075
- removed F1: 72V/0.25A, SparkFun-Fuses:PTH
- removed J1: (no value), SparkFun-Connectors:USB-C-16P
- removed J2: AVR_SPI_PROG_3X2NS, SparkFun-Connectors:2X3-NS
- removed J3: (no value), SparkFun-Connectors:1X04
- removed R1: 1.5k, adafruit:0207/7
- removed R2, R3: 75R, adafruit:0207/7
- removed R4: 10k, adafruit:0207/5V
- removed R5, R6: I2C, adafruit:0207/5V
- removed R7, R8: (no value), adafruit:0207/5V
- removed S1, S2: MOMENTARY-SWITCH-SPST-PTH-6.0MM, SparkFun-Switches:TACTILE_SWITCH_PTH_6.0MM
- removed SJ1, SJ2: (no value), jumper:SJ
- removed U2: 328P, SparkFun-IC-Microcontroller:DIP28
- removed Y1: 16MHz, SparkFun-Clocks:HC49US
- added D46, D47, D48, D49, D50, D51, D52, D53, D54, D55, D56, D57, D58, D59, D60, D61, D62, D63, D64, D65, D66, D67, D68, D69, D70, D71, D72, D73, D74, D75: (no value), adafruit:DO-1N4148
- added LED10, LED11, LED12, LED13, LED14, LED3, LED4, LED5, LED6, LED7, LED8, LED9: WS2812B, SparkFun-LED:WS2812B
- added U$41, U$42, U$43, U$44, U$45, U$46, U$47, U$48, U$49, U$50, U$51, U$52, U$53, U$54, U$55, U$56, U$57, U$58, U$59, U$60, U$61, U$62, U$63, U$64, U$65, U$66, U$67, U$68, U$69, U$70, U$71, U$72, U$73, U$74, U$75: CHERRY-MX1A-E1NW-LED, my_parts:CHERRYMX-NN-LED
- added _1: TEENSY, teensy:TEENSY
- D41, D42, D43: value WS2812B -> (none); device SparkFun-LED:WS2812B -> adafruit:DO-1N4148
- D44, D45: value 3.6V -> (none); device adafruit:DO41-7 -> adafruit:DO-1N4148
- LED1, LED2: value (none) -> WS2812B; device adafruit:LED3MM -> SparkFun-LED:WS2812B
- moved U$11 255.3 mm to (50.8, 127.0)
- moved U$12 255.3 mm to (76.2, 127.0)
- moved U$13 255.3 mm to (101.6, 127.0)
- moved U$14 255.3 mm to (127.0, 127.0)
- moved U$15 255.3 mm to (152.4, 127.0)
- moved D11 249.2 mm to (44.5, 142.9)
- moved D13 249.2 mm to (95.2, 142.9)
- moved D14 249.2 mm to (120.7, 142.9)
- moved D15 249.2 mm to (146.1, 142.9)
- moved D12 249.2 mm to (69.8, 142.9)
- moved LED1 226.5 mm to (-165.1, 88.9), flipped to the bottom
- moved LED2 223.8 mm to (-165.1, 63.5), flipped to the bottom, turned to 180 degrees
- moved D41 222.5 mm to (50.8, 142.9), flipped to the top, turned to 90 degrees
- moved D42 173.7 mm to (76.2, 142.9), flipped to the top, turned to 90 degrees
- moved U$22 129.5 mm to (-50.8, 101.6)
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Connections:
- removed net I2C_SCL: J3.2, R5.1, SJ1.1, U2.28
- removed net I2C_SDA: J3.3, R6.1, SJ2.1, U2.27
- removed net N$43: F1.P$2, J1.VBUS1, J1.VBUS2
- removed net N$44: D44.C, J1.A7, J1.B7, R1.2, R3.2
- removed net N$45: U2.2
- removed net RESET: J2.5, R4.1, S1.3, U2.1
- removed net RGB: LED1.K, LED2.K
- removed net USB_D+: R2.1, U2.4
- removed net USB_D-: R3.1, U2.5
- new net COLUMN10: D11.C, D26.C, D41.C, D56.C, D71.C, _1.D7
- new net COLUMN11: D12.C, D27.C, D42.C, D57.C, D72.C, _1.B4
- new net COLUMN12: D13.C, D28.C, D43.C, D58.C, D73.C, _1.B5
- new net COLUMN13: D14.C, D29.C, D44.C, D59.C, D74.C, _1.B6
- new net COLUMN14: D15.C, D30.C, D45.C, D60.C, D75.C, _1.F7
- new net N$113: _1.REF
- new net N$114: _1.F0
- new net N$115: _1.F1
- new net N$116: _1.F4
- new net N$117: _1.F5
- new net N$120: _1.5V2
- new net N$121: _1.RST
- new net N$122: _1.GRND1
- new net N$54: D41.A, U$41.SIDE
- new net N$55: D42.A, U$42.SIDE
- new net N$56: D43.A, U$43.SIDE
- new net N$57: D44.A, U$44.SIDE
- new net N$58: D45.A, U$45.SIDE
- new net N$59: D46.A, U$46.SIDE
- new net N$60: D47.A, U$47.SIDE
- new net N$61: D48.A, U$48.SIDE
- new net N$62: D49.A, U$49.SIDE
- new net N$63: D50.A, U$50.SIDE
- new net N$64: D51.A, U$51.SIDE
- new net N$65: D52.A, U$52.SIDE
- new net N$66: D53.A, U$53.SIDE
- new net N$67: D54.A, U$54.SIDE
- new net N$68: D55.A, U$55.SIDE
- new net N$69: D56.A, U$56.SIDE
- new net N$70: D57.A, U$57.SIDE
- new net N$71: D58.A, U$58.SIDE
- new net N$72: D59.A, U$59.SIDE
- new net N$73: D60.A, U$60.SIDE
- new net N$74: D61.A, U$61.SIDE
- new net N$75: D62.A, U$62.SIDE
- new net N$76: D63.A, U$63.SIDE
- new net N$77: D64.A, U$64.SIDE
- new net N$78: D65.A, U$65.SIDE
- new net N$79: D66.A, U$66.SIDE
- new net N$80: D67.A, U$67.SIDE
- new net N$81: D68.A, U$68.SIDE
- new net N$82: D69.A, U$69.SIDE
- new net N$83: D70.A, U$70.SIDE
- new net N$84: D71.A, U$71.SIDE
- new net N$85: D72.A, U$72.SIDE
- new net N$86: D73.A, U$73.SIDE
- new net N$87: D74.A, U$74.SIDE
- new net N$88: D75.A, U$75.SIDE
- new net N$89: LED11.2, LED12.4
- new net N$90: LED12.2, LED13.4
- new net N$91: LED13.2, LED14.4
- new net ROW4: U$61.UP, U$62.UP, U$63.UP, U$64.UP, U$65.UP, U$66.UP, U$67.UP, U$68.UP, U$69.UP, U$70.UP, U$71.UP, U$72.UP, U$73.UP, U$74.UP, U$75.UP
- net 5V: now also LED1.3, LED10.3, LED11.3, LED12.3, LED13.3, LED14.3, LED2.3, LED3.3, LED4.3, LED5.3, LED6.3, LED7.3, LED8.3, LED9.3, _1.+5V; no longer C1.+, C2.1, C3.1, D41.3, D42.3, D43.3, F1.P$1, J2.2, J3.1, R1.1, R4.2, R5.2, R6.2
- net COLUMN0: now also D16.C, D46.C, D61.C, _1.B7; no longer D11.C, D21.C, U2.14
- net COLUMN1: now also D17.C, D47.C, D62.C, _1.D0; no longer D12.C, D22.C
- net COLUMN2: now also D18.C, D48.C, D63.C, _1.D1; no longer D13.C, D23.C
- net COLUMN3: now also D19.C, D49.C, D64.C, _1.D2; no longer D14.C, D24.C, S2.1, U2.11
- net COLUMN4: now also D20.C, D50.C, D65.C, _1.D3; no longer D15.C, D25.C, U2.16
- net COLUMN5: now also D21.C, D51.C, D66.C, _1.C6; no longer D16.C, D26.C, U2.15
- net COLUMN6: now also D22.C, D52.C, D67.C, _1.C7; no longer D17.C, D27.C, U2.23
- net COLUMN7: now also D23.C, D53.C, D68.C, _1.D5; no longer D18.C, D28.C, U2.24
- net COLUMN8: now also D24.C, D54.C, D69.C, _1.D4; no longer D19.C, D29.C, U2.25
- net COLUMN9: now also D25.C, D55.C, D70.C, _1.D6; no longer D20.C, D30.C, U2.26
- net GND: now also LED1.1, LED10.1, LED11.1, LED12.1, LED13.1, LED14.1, LED2.1, LED3.1, LED4.1, LED5.1, LED6.1, LED7.1, LED8.1, LED9.1, U$41.LED-, U$42.LED-, U$43.LED-, U$44.LED-, U$45.LED-, U$46.LED-, U$47.LED-, U$48.LED-, U$49.LED-, U$50.LED-, U$51.LED-, U$52.LED-, U$53.LED-, U$54.LED-, U$55.LED-, U$56.LED-, U$57.LED-, U$58.LED-, U$59.LED-, U$60.LED-, U$61.LED-, U$62.LED-, U$63.LED-, U$64.LED-, U$65.LED-, U$66.LED-, U$67.LED-, U$68.LED-, U$69.LED-, U$70.LED-, U$71.LED-, U$72.LED-, U$73.LED-, U$74.LED-, U$75.LED-, _1.GND; no longer C1.-, C2.2, C3.2, C4.1, C5.1, D41.1, D42.1, D43.1, D44.A, D45.A, J1.GND, J1.GND2, J2.6, J3.4, S1.1, S2.3
- net LED+: now also U$41.LED+, U$42.LED+, U$43.LED+, U$44.LED+, U$45.LED+, U$46.LED+, U$47.LED+, U$48.LED+, U$49.LED+, U$50.LED+, U$51.LED+, U$52.LED+, U$53.LED+, U$54.LED+, U$55.LED+, U$56.LED+, U$57.LED+, U$58.LED+, U$59.LED+, U$60.LED+, U$61.LED+, U$62.LED+, U$63.LED+, U$64.LED+, U$65.LED+, U$66.LED+, U$67.LED+, U$68.LED+, U$69.LED+, U$70.LED+, U$71.LED+, U$72.LED+, U$73.LED+, U$74.LED+, U$75.LED+
- net N$41: now also LED1.2, LED2.4; no longer D41.2, D42.4
- net N$42: now also LED2.2, LED3.4; no longer D42.2, D43.4
- net N$46: now also LED3.2, LED4.4; no longer D45.C, J1.A6, J1.B6, R2.2
- net N$47: now also LED4.2, LED5.4; no longer C5.2, U2.10, Y1.1
- net N$48: now also LED5.2, LED6.4; no longer C4.2, U2.9, Y1.2
- net N$49: now also LED6.2, LED7.4; no longer R7.1, SJ1.2
- net N$50: now also LED7.2, LED8.4; no longer U2.3
- net N$51: now also LED8.2, LED9.4; no longer LED1.A, R7.2
- net N$52: now also LED10.4, LED9.2; no longer R8.1, SJ2.2
- net N$53: now also LED10.2, LED11.4; no longer LED2.A, R8.2
- net RGB_DATA: now also LED1.4, _1.F6; no longer D41.4, U2.12
- net ROW0: now also U$11.UP, U$12.UP, U$13.UP, U$14.UP, U$15.UP, _1.B0; no longer J2.1, U2.18
- net ROW1: now also U$21.UP, U$22.UP, U$23.UP, U$24.UP, U$25.UP, U$26.UP, U$27.UP, U$28.UP, U$29.UP, U$30.UP, _1.B1; no longer J2.3, U$11.UP, U$12.UP, U$13.UP, U$14.UP, U$15.UP, U2.19
- net ROW2: now also U$31.UP, U$32.UP, U$33.UP, U$34.UP, U$35.UP, U$36.UP, U$37.UP, U$38.UP, U$39.UP, U$40.UP, U$41.UP, U$42.UP, U$43.UP, U$44.UP, U$45.UP, _1.B2; no longer J2.4, U$21.UP, U$22.UP, U$23.UP, U$24.UP, U$25.UP, U$26.UP, U$27.UP, U$28.UP, U$29.UP, U$30.UP, U2.17
- net ROW3: now also U$46.UP, U$47.UP, U$48.UP, U$49.UP, U$50.UP, U$51.UP, U$52.UP, U$53.UP, U$54.UP, U$55.UP, U$56.UP, U$57.UP, U$58.UP, U$59.UP, U$60.UP, _1.B3; no longer U$31.UP, U$32.UP, U$33.UP, U$34.UP, U$35.UP, U$36.UP, U$37.UP, U$38.UP, U$39.UP, U$40.UP, U2.6
Routing:
- net LED+: track 1057.8 -> 2032.1 mm
- net GND: track 1221.3 -> 2181.0 mm, vias 1 -> 3
- net COLUMN1: track 9.73 -> 396.7 mm, vias 0 -> 1
- net COLUMN2: track 9.75 -> 366.1 mm
- net ROW4: track 0.00 -> 355.6 mm
- net ROW2: track 280.2 -> 499.1 mm, vias 2 -> 9
- net ROW3: track 302.8 -> 485.6 mm, vias 0 -> 1
- net RGB_DATA: track 222.3 -> 386.4 mm, vias 2 -> 5
- net ROW0: track 316.0 -> 466.3 mm, vias 1 -> 2
- net COLUMN10: track 0.00 -> 140.5 mm, vias 0 -> 1
- net N$88: track 0.00 -> 134.5 mm, vias 0 -> 1
- net N$82: track 0.00 -> 129.2 mm
- net N$75: track 0.00 -> 125.8 mm
- net N$76: track 0.00 -> 125.1 mm
- net 5V: track 346.0 -> 470.1 mm, vias 5 -> 6
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Other:
- board size 279.4 x 114.3 mm -> 406.4 x 139.7 mm
- board text removed: "A 40 key macropad"
- board text removed: "Designed and assembled in Hannover"
- board text removed: "The Extender"
- board text removed: "by Carlos Rödiger"
- board text removed: "powered by the QMK Firmware"

Commit message: The first release
This is what you might call the first release. I will order some prototype PCBs with propably a few minor tweeks!
Parts:
- removed _1: TEENSY, teensy:TEENSY
- added C1, C2: 22p, adafruit:C025-025X050
- added C3, C4: 0.1u, adafruit:C025-025X050
- added C5: 4.7u, adafruit:E2-4
- added D76, D77: (no value), diode:DO34Z7
- added F1: 72V/0.25A, SparkFun-Fuses:PTH
- added IC1: ATMEGA32A-PU, ATMEGA32A-PU:DIP1556W56P254L5232H483Q40N
- added ISP1: AVRISP-6, adafruit:AVRISP
- added J1: USB4085-GF-A_REVA, USB4085-GF-A_REVA:GCT_USB4085-GF-A_REVA
- added LED15: (no value), adafruit:LED3MM
- added R1: 10k, adafruit:0207/9
- added R2, R7: 1.5k, adafruit:0207/9
- added R3, R4: 5.1k, adafruit:0207/9
- added R5, R6: 75R, adafruit:0207/9
- added S1, S2: (no value), SparkFun-Retired:TACTILE-PTH
- added X1: 49S/18PF, Crystals:XTAL_HC49
Connections:
- removed net N$113: _1.REF
- removed net N$114: _1.F0
- removed net N$115: _1.F1
- removed net N$116: _1.F4
- removed net N$117: _1.F5
- removed net N$120: _1.5V2
- removed net N$121: _1.RST
- removed net N$122: _1.GRND1
- new net BOOT: IC1.18, S2.3
- new net LED-: U$1.LED-, U$10.LED-, U$11.LED-, U$12.LED-, U$13.LED-, U$14.LED-, U$15.LED-, U$16.LED-, U$17.LED-, U$18.LED-, U$19.LED-, U$2.LED-, U$20.LED-, U$21.LED-, U$22.LED-, U$23.LED-, U$24.LED-, U$25.LED-, U$26.LED-, U$27.LED-, U$28.LED-, U$29.LED-, U$3.LED-, U$30.LED-, U$31.LED-, U$32.LED-, U$33.LED-, U$34.LED-, U$35.LED-, U$36.LED-, U$37.LED-, U$38.LED-, U$39.LED-, U$4.LED-, U$40.LED-, U$41.LED-, U$42.LED-, U$43.LED-, U$44.LED-, U$45.LED-, U$46.LED-, U$47.LED-, U$48.LED-, U$49.LED-, U$5.LED-, U$50.LED-, U$51.LED-, U$53.LED-, U$54.LED-, U$55.LED-, U$56.LED-, U$57.LED-, U$58.LED-, U$59.LED-, U$6.LED-, U$60.LED-, U$61.LED-, U$62.LED-, U$63.LED-, U$64.LED-, U$65.LED-, U$66.LED-, U$67.LED-, U$68.LED-, U$69.LED-, U$7.LED-, U$71.LED-, U$72.LED-, U$73.LED-, U$74.LED-, U$75.LED-, U$8.LED-, U$9.LED-
- new net LED-\: U$70.LED-
- new net MISO: IC1.7, ISP1.1
- new net MOSI: IC1.6, ISP1.4
- new net N$119: U$52.LED-
- new net N$43: C1.2, IC1.12, X1.2
- new net N$44: C2.2, IC1.13, X1.1
- new net N$45: LED15.K, R2.1
- new net N$92: J1.A1, J1.A12, J1.B1, J1.B12
- new net N$93: F1.P$2, J1.A4, J1.A9, J1.B4, J1.B9
- new net N$94: J1.P1, J1.P2, J1.P3, J1.P4
- new net N$95: J1.A5, R3.1
- new net N$96: D76.C, J1.A7, J1.B7, R5.1, R7.1
- new net N$97: D77.C, J1.A6, J1.B6, R6.1
- new net N$98: J1.B5, R4.1
- new net RESET: IC1.9, ISP1.5, R1.1, S1.3
- new net SCK: IC1.8, ISP1.3
- new net USB_D+: IC1.16, R6.2
- new net USB_D-: IC1.17, R5.2
- net 5V: now also C3.1, C4.1, C5.+, F1.P$1, IC1.10, IC1.30, ISP1.2, LED15.A, R1.2, R7.2; no longer _1.+5V
- net COLUMN0: now also IC1.14; no longer _1.B7
- net COLUMN1: now also IC1.15; no longer _1.D0
- net COLUMN10: now also IC1.34; no longer _1.D7
- net COLUMN11: now also IC1.33; no longer _1.B4
- net COLUMN12: now also IC1.32; no longer _1.B5
- net COLUMN13: now also IC1.29; no longer _1.B6
- net COLUMN14: now also IC1.28; no longer _1.F7
- net COLUMN2: now also IC1.19; no longer _1.D1
- net COLUMN3: now also IC1.20; no longer _1.D2
- net COLUMN4: now also IC1.40; no longer _1.D3
- net COLUMN5: now also IC1.39; no longer _1.C6
- net COLUMN6: now also IC1.38; no longer _1.C7
- net COLUMN7: now also IC1.37; no longer _1.D5
- net COLUMN8: now also IC1.36; no longer _1.D4
- net COLUMN9: now also IC1.35; no longer _1.D6
- net GND: now also C1.1, C2.1, C3.2, C4.2, C5.-, D76.A, D77.A, IC1.11, IC1.31, ISP1.6, R2.2, R3.2, R4.2, S1.1, S2.1; no longer U$1.LED-, U$10.LED-, U$11.LED-, U$12.LED-, U$13.LED-, U$14.LED-, U$15.LED-, U$16.LED-, U$17.LED-, U$18.LED-, U$19.LED-, U$2.LED-, U$20.LED-, U$21.LED-, U$22.LED-, U$23.LED-, U$24.LED-, U$25.LED-, U$26.LED-, U$27.LED-, U$28.LED-, U$29.LED-, U$3.LED-, U$30.LED-, U$31.LED-, U$32.LED-, U$33.LED-, U$34.LED-, U$35.LED-, U$36.LED-, U$37.LED-, U$38.LED-, U$39.LED-, U$4.LED-, U$40.LED-, U$41.LED-, U$42.LED-, U$43.LED-, U$44.LED-, U$45.LED-, U$46.LED-, U$47.LED-, U$48.LED-, U$49.LED-, U$5.LED-, U$50.LED-, U$51.LED-, U$52.LED-, U$53.LED-, U$54.LED-, U$55.LED-, U$56.LED-, U$57.LED-, U$58.LED-, U$59.LED-, U$6.LED-, U$60.LED-, U$61.LED-, U$62.LED-, U$63.LED-, U$64.LED-, U$65.LED-, U$66.LED-, U$67.LED-, U$68.LED-, U$69.LED-, U$7.LED-, U$70.LED-, U$71.LED-, U$72.LED-, U$73.LED-, U$74.LED-, U$75.LED-, U$8.LED-, U$9.LED-, _1.GND
- net RGB_DATA: now also IC1.27; no longer _1.F6
- net ROW0: now also IC1.1; no longer _1.B0
- net ROW1: now also IC1.2; no longer _1.B1
- net ROW2: now also IC1.3; no longer _1.B2
- net ROW3: now also IC1.4; no longer _1.B3
- net ROW4: now also IC1.5
Routing:
- net LED-: track 0.00 -> 2105.0 mm, vias 0 -> 2
- net GND: track 2181.0 -> 604.5 mm, vias 3 -> 4
- net COLUMN4: track 305.4 -> 474.2 mm
- net LED+: track 2032.1 -> 2172.6 mm
- net COLUMN0: track 404.3 -> 535.5 mm
- net 5V: track 470.1 -> 584.1 mm, vias 6 -> 4
- net COLUMN1: track 396.7 -> 503.2 mm, vias 1 -> 2
- net RGB_DATA: track 386.4 -> 487.5 mm, vias 5 -> 2
- net ROW4: track 355.6 -> 454.1 mm
- net COLUMN2: track 366.1 -> 458.3 mm
- net COLUMN13: track 55.8 -> 137.3 mm, vias 1 -> 2
- net ROW1: track 456.8 -> 534.6 mm, vias 11 -> 13
- net COLUMN10: track 140.5 -> 217.5 mm, vias 1 -> 3
- net USB_D-: track 0.00 -> 69.7 mm
- net RESET: track 0.00 -> 69.5 mm
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Other:
- board size 406.4 x 139.7 mm -> 419.1 x 139.7 mm

Commit message: This is the first prototype version.
I made quite a few tweeks to the PCB, a lot of traces were redrawn or moved.
Parts:
- flipped D2 to the top
Routing:
- net LED+: track 2172.6 -> 2108.8 mm
- net N$66: track 128.0 -> 101.2 mm
- net N$70: track 117.0 -> 100.2 mm
- net RGB_DATA: track 487.5 -> 471.8 mm
- net N$55: track 86.7 -> 71.1 mm
- net COLUMN4: track 474.2 -> 461.1 mm
- net COLUMN3: track 388.5 -> 375.6 mm
- net COLUMN0: track 535.5 -> 523.0 mm
- net RESET: track 69.5 -> 58.2 mm
- net COLUMN1: track 503.2 -> 493.9 mm
- net N$31: track 72.9 -> 64.7 mm
- net COLUMN2: track 458.3 -> 450.4 mm
- net COLUMN6: track 277.8 -> 271.1 mm
- net COLUMN13: track 137.3 -> 131.2 mm
- net COLUMN5: track 309.0 -> 303.5 mm
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Other:
- board text added: "JLCJLCJLCJLC"
- board text added: "The Extender (5x15 keys) Powered by QMK Firmware by Carlos Rödiger designed and manufactured in Hanover, Germany Version V0.1"
- board text added: "https://github.com/FrancTheCat/The-Extender"
