File: PCB Files/Rev 2/Order.brd (EAGLE design)
At the start: 410 x 140 mm, 186 parts, among them IC1 ATMEGA32A-PU, J1 USB4085-GF-A_REVA, X1 49S/18PF

Commit message: I am stupid
I changed the spacing between the keys to the right dimension (19mm) and rearanhged the keyboard. I also added a rotary encoder and a DIP switch.
Parts:
- added SW1: EC12E_SW, switch-alps:ALPS_EC12E_SW
- added SW2: (no value), special:EDG-04
- moved LED15 117.0 mm to (292.0, 92.0)
- moved S2 108.2 mm to (297.0, 32.0)
- moved ISP1 106.3 mm to (292.0, 72.0), turned to 180 degrees
- moved R7 104.0 mm to (290.0, 108.0)
- moved R4 103.9 mm to (290.0, 105.0)
- moved R3 103.9 mm to (290.0, 102.0)
- moved R1 100.4 mm to (291.0, 28.0)
- moved S1 100.3 mm to (297.0, 24.0)
- moved R2 99.4 mm to (313.0, 96.0)
- moved R5 99.3 mm to (310.0, 96.0)
- moved J1 99.2 mm to (306.0, 108.0)
- moved R6 99.1 mm to (307.0, 96.0)
- moved D77 98.9 mm to (304.0, 96.0)
- moved D76 98.6 mm to (302.0, 96.0)
- moved C3 97.8 mm to (299.0, 97.0)
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Connections:
- new net ENCODER_A: IC1.25, SW1.A
- new net ENCODER_B: IC1.26, SW1.B
- new net N$100: IC1.23, SW2.6
- new net N$101: IC1.22, SW2.7
- new net N$102: IC1.21, SW2.8
- new net N$99: IC1.24, SW2.5
- net GND: now also SW1.C, SW2.1, SW2.2, SW2.3, SW2.4
Routing:
- net LED+: track 2177.7 -> 0.00 mm
- net LED-: track 2115.1 -> 0.00 mm, vias 2 -> 0
- net GND: track 775.0 -> 0.00 mm, vias 2 -> 0
- net ROW1: track 687.4 -> 0.00 mm, vias 5 -> 0
- net 5V: track 611.4 -> 0.00 mm, vias 8 -> 0
- net ROW0: track 531.2 -> 0.00 mm
- net ROW2: track 521.1 -> 0.00 mm, vias 3 -> 0
- net ROW4: track 515.3 -> 0.00 mm
- net ROW3: track 463.2 -> 0.00 mm, vias 3 -> 0
- net COLUMN0: track 449.7 -> 0.00 mm
- net COLUMN1: track 429.2 -> 0.00 mm
- net COLUMN2: track 420.7 -> 0.00 mm, vias 4 -> 0
- net RGB_DATA: track 412.5 -> 0.00 mm
- net COLUMN3: track 379.3 -> 0.00 mm, vias 4 -> 0
- net COLUMN4: track 321.4 -> 0.00 mm, vias 1 -> 0
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Other:
- board size 410 x 140 mm -> 324 x 111 mm

Commit message: now with Traces!
I added the traces to the new, now less stupid PCB.
Parts:
- moved D1 12.0 mm to (16.0, 104.0)
- moved D10 12.0 mm to (187.0, 104.0)
- moved D11 12.0 mm to (206.0, 104.0)
- moved D12 12.0 mm to (225.0, 104.0)
- moved D13 12.0 mm to (244.0, 104.0)
- moved D14 12.0 mm to (263.0, 104.0)
- moved D15 12.0 mm to (282.0, 104.0)
- moved D2 12.0 mm to (35.0, 104.0)
- moved D3 12.0 mm to (54.0, 104.0)
- moved D4 12.0 mm to (73.0, 104.0)
- moved D5 12.0 mm to (92.0, 104.0)
- moved D6 12.0 mm to (111.0, 104.0)
- moved D61 12.0 mm to (4.00, 104.0)
- moved D62 12.0 mm to (23.0, 104.0)
- moved D63 12.0 mm to (42.0, 104.0)
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Connections:
- removed net LED-\: U$70.LED-
- removed net N$119: U$52.LED-
- net LED-: now also U$52.LED-, U$70.LED-
Routing:
- net LED-: track 0.00 -> 1500.3 mm
- net LED+: track 0.00 -> 1489.7 mm
- net GND: track 0.00 -> 533.3 mm, vias 0 -> 1
- net 5V: track 0.00 -> 403.8 mm, vias 0 -> 1
- net ROW4: track 0.00 -> 366.0 mm
- net ROW3: track 0.00 -> 346.3 mm
- net COLUMN0: track 0.00 -> 332.9 mm, vias 0 -> 1
- net ROW2: track 0.00 -> 325.2 mm
- net COLUMN1: track 0.00 -> 321.8 mm
- net COLUMN2: track 0.00 -> 306.3 mm, vias 0 -> 1
- net ROW1: track 0.00 -> 303.7 mm
- net RGB_DATA: track 0.00 -> 301.1 mm, vias 0 -> 2
- net COLUMN3: track 0.00 -> 293.0 mm
- net ROW0: track 0.00 -> 288.1 mm
- net COLUMN4: track 0.00 -> 248.8 mm
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