File: PCB Files/Rev 2/Order.brd (EAGLE design)
At the start: 324 x 111 mm, 188 parts, among them IC1 ATMEGA32A-PU, J1 USB4085-GF-A_REVA, SW1 EC12E_SW, X1 49S/18PF

Commit message: new LED placement
Parts:
- added LED16: WS2812B, SparkFun-LED:WS2812B
- added LED17: (no value), adafruit:LED3MM
- LED15: value (none) -> WS2812B; device adafruit:LED3MM -> SparkFun-LED:WS2812B
- moved LED15 72.8 mm to (285.5, 19.5), flipped to the bottom
- moved LED1 19.5 mm to (19.5, 19.5)
- moved LED10 19.0 mm to (190.0, 19.5)
- moved LED11 19.0 mm to (209.5, 19.5)
- moved LED12 19.0 mm to (228.5, 19.5)
- moved LED13 19.0 mm to (247.5, 19.5)
- moved LED14 19.0 mm to (266.5, 19.5)
- moved LED2 19.0 mm to (38.5, 19.5)
- moved LED3 19.0 mm to (57.5, 19.5)
- moved LED4 19.0 mm to (76.5, 19.5)
- moved LED5 19.0 mm to (95.5, 19.5)
- moved LED6 19.0 mm to (114.5, 19.5)
- moved LED7 19.0 mm to (133.5, 19.5)
- moved LED8 19.0 mm to (152.5, 19.5)
- moved LED9 19.0 mm to (171.5, 19.5)
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Connections:
- new net N$103: LED15.2, LED16.4
- new net N$104: LED14.2, LED15.4
- net 5V: now also LED15.3, LED16.3, LED17.A; no longer LED15.A
- net GND: now also LED15.1, LED16.1
- net N$45: now also LED17.K; no longer LED15.K
Routing:
- net 5V: track 403.8 -> 480.4 mm, vias 1 -> 5
- net GND: track 533.3 -> 587.3 mm
- net RGB_DATA: track 301.1 -> 339.8 mm, vias 2 -> 0
- net N$103: track 0.00 -> 25.5 mm
- net N$104: track 0.00 -> 19.1 mm, vias 0 -> 2
- net ENCODER_A: track 53.0 -> 59.3 mm
- net ENCODER_B: track 53.8 -> 57.4 mm
- net BOOT: track 11.0 -> 9.12 mm
- net RESET: track 62.5 -> 61.1 mm
- net N$99: track 16.3 -> 15.2 mm
- net N$41: track 14.4 -> 15.4 mm
- net N$100: track 14.5 -> 13.8 mm
- net COLUMN2: track 306.3 -> 307.0 mm
- net N$53: track 15.2 -> 15.8 mm
- net N$52: track 15.2 -> 14.7 mm
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
Commit message: Added to QMK badge
The QMK badge will now be etched to the underside in cooper. I also removed to soldermask to it should look nice and shiny!
Routing:
- net N$84: track 90.2 -> 93.2 mm
- net N$79: track 90.2 -> 93.2 mm
- net N$88: track 90.2 -> 93.2 mm
- net GND: track 587.3 -> 588.5 mm
Other:
- board text added: "A quick tip: the distance between two switches is 19mm, not 1"! (I wasted 35 Euros on this...)"
